File: Embebidos_2019/Embebidos_2019.sch (KiCad schematic (older format))
At the start: 0 parts

Commit message: Add files via upload
Changed lines of the file:
@@
 F5 "ADS_CLKSEL" I L 7250 5900 50
 F6 "ADS_DRDY" I L 7250 6100 50
-F7 "SPI_ADS(3..0)" B L 7250 5800 50
-F8 "AVDD" I L 7250 6500 50
-F9 "AVSS" I L 7250 6650 50
+F7 "AVDD" I L 7250 6500 50
+F8 "AVSS" I L 7250 6650 50
+F9 "SPI_ADS[3..0]" B L 7250 5800 50
 $EndSheet
 $Sheet
@@
 F4 "USART_TX" O L 7250 4250 50
 F5 "BOOT0" O L 7250 3800 50
-F6 "SPI_OM_(3..0)" B L 7250 4400 50
-F7 "I2C_OM(1..0)" B L 7250 4600 50
-F8 "JTAG_OM(5..0)" B L 7250 4800 50
+F6 "SPI_OM_[3..0]" B L 7250 4600 50
+F7 "I2C_OM[1..0]" B L 7250 4800 50
+F8 "JTAG_OM[5..0]" B L 7250 4400 50
 $EndSheet
 $Sheet
@@
 F2 "BOOT0" I R 5400 3300 50
 F3 "BOOT1" I R 5400 3400 50
-F4 "JTAG(5..0)" B R 5400 4150 50
-F5 "SPI2_U(3..0)" B R 5400 4350 50
-F6 "UART_CTS" I R 5400 2450 50
-F7 "UART1_RX" I R 5400 2950 50
-F8 "UART1_TX" O R 5400 2800 50
-F9 "UART2_RX" I R 5400 3700 50
-F10 "UART2_TX" O R 5400 3550 50
-F11 "UART_RTS" O R 5400 2650 50
-F12 "SPI1_U(3..0)" B R 5400 3850 50
-F13 "A_CLKSEL" O R 5400 4500 50
-F14 "A_CLK" O R 5400 4650 50
-F15 "A_START" O R 5400 4950 50
-F16 "A_PWDN" O R 5400 5100 50
-F17 "A_DRY" O R 5400 4800 50
-F18 "BL_WAKE" O R 5400 3100 50
-F19 "I2C_U(1..0)" B R 5400 4000 50
+F4 "UART_CTS" I R 5400 2450 50
+F5 "UART1_RX" I R 5400 2950 50
+F6 "UART1_TX" O R 5400 2800 50
+F7 "UART2_RX" I R 5400 3700 50
+F8 "UART2_TX" O R 5400 3550 50
+F9 "UART_RTS" O R 5400 2650 50
+F10 "A_CLKSEL" O R 5400 4500 50
+F11 "A_CLK" O R 5400 4650 50
+F12 "A_START" O R 5400 4950 50
+F13 "A_PWDN" O R 5400 5100 50
+F14 "A_DRY" O R 5400 4800 50
+F15 "BL_WAKE" O R 5400 3100 50
+F16 "JTAG[5..0]" B R 5400 3850 50
+F17 "SPI2_U[3..0]" B R 5400 4000 50
+F18 "SPI1_U[3..0]" B R 5400 4350 50
+F19 "I2C_U[1..0]" B R 5400 4150 50
 $EndSheet
 Wire Wire Line

Commit message: Add files via upload
Changed lines of the file:
@@
 F6 "SPI_OM_[3..0]" B L 7250 4600 50
 F7 "I2C_OM[1..0]" B L 7250 4800 50
-F8 "JTAG_OM[5..0]" B L 7250 4400 50
+F8 "JTAGOM[5..0]" B L 7250 4400 50
 $EndSheet
 $Sheet
@@
 F15 "BL_WAKE" O R 5400 3100 50
 F16 "JTAG[5..0]" B R 5400 3850 50
-F17 "SPI2_U[3..0]" B R 5400 4000 50
-F18 "SPI1_U[3..0]" B R 5400 4350 50
-F19 "I2C_U[1..0]" B R 5400 4150 50
+F17 "SPI2_U[3..0]" B R 5400 4350 50
+F18 "SPI1_U[3..0]" B R 5400 4000 50
+F19 "I2C1_U[1..0]" B R 5400 4150 50
 $EndSheet
 Wire Wire Line
