File: Embebidos_2019/BLUETOOTH.sch (KiCad schematic (older format))
At the start: 5 parts, among them J1 A106614-ND

Commit message: Add files via upload
Changed lines of the file:
@@
 Wire Wire Line
 	4250 3400 4800 3400
-Wire Wire Line
-	1500 3200 1650 3200
-Wire Wire Line
-	950  3200 1650 3200
 $Comp
 L BAT2032:C C58
@@
 	3350 2700 3350 2900
 Wire Wire Line
-	3250 2250 3250 2900
+	3250 2250 3250 2500
 $Comp
 L BAT2032:C C57
@@
 Wire Wire Line
 	3300 2250 3350 2250
+Wire Wire Line
+	1500 3200 1650 3200
+Wire Wire Line
+	950  3200 1650 3200
+$Comp
+L power:PWR_FLAG #FLG0103
+U 1 1 5CEFFD9E
+P 3050 2500
+F 0 "#FLG0103" H 3050 2575 50  0001 C CNN
+F 1 "PWR_FLAG" V 3050 2627 50  0000 L CNN
+F 2 "" H 3050 2500 50  0001 C CNN
+F 3 "~" H 3050 2500 50  0001 C CNN
+	1    3050 2500
+	0    -1   -1   0
+$EndComp
+Wire Wire Line
+	3050 2500 3250 2500
+Connection ~ 3250 2500
+Wire Wire Line
+	3250 2500 3250 2900
 $EndSCHEMATC

Commit message: Add files via upload
Parts:
- J1: footprint Connector_PinSocket_2.54mm:PinSocket_1x12_P2.54mm_Vertical -> Connector_PinHeader_2.54mm:PinHeader_2x06_P2.54mm_Vertical
Changed lines of the file:
@@
 F 0 "J1" H 2908 6531 50  0000 C CNN
 F 1 "A106614-ND" H 2908 6440 50  0000 C CNN
-F 2 "Connector_PinSocket_2.54mm:PinSocket_1x12_P2.54mm_Vertical" H 2800 5850 50  0001 C CNN
+F 2 "Connector_PinHeader_2.54mm:PinHeader_2x06_P2.54mm_Vertical" H 2800 5850 50  0001 C CNN
 F 3 "~" H 2800 5850 50  0001 C CNN
 	1    2800 5850

Commit message: Add files via upload
Parts:
- removed J1: A106614-ND, Connector_PinHeader_2.54mm:PinHeader_2x06_P2.54mm_Vertical, symbol Connector:Conn_01x12_Male
Connections:
- net AIO0: no longer names the net of MOD1.5 (AIO_0)
- net AIO1: no longer names the net of MOD1.4 (AIO_1)
- net AIO2: no longer names the net of MOD1.3 (AIO_2)
- net PIO10: no longer names the net of MOD1.28 (PIO_10)
- net PIO11: no longer names the net of MOD1.29 (PIO_11)
- net PIO3: no longer names the net of MOD1.8 (PIO_3)
- net PIO4: no longer names the net of MOD1.9 (PIO_4)
- net PIO7: no longer names the net of MOD1.14 (PIO_6/SPI_MOSI)
- net PIO8: no longer names the net of MOD1.19 (PIO_8)
- net PIO9: no longer names the net of MOD1.26 (PIO_9)
- no-connect marks 4 -> 14
Changed lines of the file:
@@
 WAKE
 Connection ~ 1650 3200
-$Comp
-L Connector:Conn_01x12_Male J1
-U 1 1 5CEDDACF
-P 2800 5850
-F 0 "J1" H 2908 6531 50  0000 C CNN
-F 1 "A106614-ND" H 2908 6440 50  0000 C CNN
-F 2 "Connector_PinHeader_2.54mm:PinHeader_2x06_P2.54mm_Vertical" H 2800 5850 50  0001 C CNN
-F 3 "~" H 2800 5850 50  0001 C CNN
-	1    2800 5850
-	1    0    0    -1
-$EndComp
-$Comp
-L power:Earth #PWR03
-U 1 1 5CEE2278
-P 3450 5350
-F 0 "#PWR03" H 3450 5100 50  0001 C CNN
-F 1 "Earth" H 3450 5200 50  0001 C CNN
-F 2 "" H 3450 5350 50  0001 C CNN
-F 3 "~" H 3450 5350 50  0001 C CNN
-	1    3450 5350
-	0    -1   -1   0
-$EndComp
-Wire Wire Line
-	3450 5350 3000 5350
-Text GLabel 3450 5450 2    50   Input ~ 0
-+3.3V_MCU
-Wire Wire Line
-	3450 5450 3000 5450
-Text Label 4500 3500 0    50   ~ 0
-PIO7
-Wire Wire Line
-	4500 3500 4250 3500
-Text Label 4500 3800 0    50   ~ 0
-PIO9
-Wire Wire Line
-	4500 3800 4250 3800
-Text Label 4500 3900 0    50   ~ 0
-PIO10
-Text Label 4500 4000 0    50   ~ 0
-PIO11
-Wire Wire Line
-	4500 3900 4250 3900
-Wire Wire Line
-	4500 4000 4250 4000
-Text Label 2300 3300 2    50   ~ 0
-AIO0
-Text Label 2300 3400 2    50   ~ 0
-AIO1
-Text Label 2300 3500 2    50   ~ 0
-AIO2
-Text Label 2300 3700 2    50   ~ 0
-PIO3
-Text Label 2300 3800 2    50   ~ 0
-PIO4
-Text Label 2300 3900 2    50   ~ 0
-PIO8
-Wire Wire Line
-	2300 3300 2550 3300
-Wire Wire Line
-	2300 3400 2550 3400
-Wire Wire Line
-	2300 3500 2550 3500
-Wire Wire Line
-	2300 3700 2550 3700
-Wire Wire Line
-	2300 3800 2550 3800
-Wire Wire Line
-	2300 3900 2550 3900
-Text Label 3500 5550 0    50   ~ 0
-AIO0
-Text Label 3500 5650 0    50   ~ 0
-AIO1
-Text Label 3500 5750 0    50   ~ 0
-AIO2
-Text Label 3500 5850 0    50   ~ 0
-PIO3
-Text Label 3500 5950 0    50   ~ 0
-PIO4
-Text Label 3500 6050 0    50   ~ 0
-PIO8
-Text Label 3500 6150 0    50   ~ 0
-PIO7
-Text Label 3500 6250 0    50   ~ 0
-PIO9
-Text Label 3500 6350 0    50   ~ 0
-PIO10
-Text Label 3500 6450 0    50   ~ 0
-PIO11
-Wire Wire Line
-	3500 5550 3000 5550
-Wire Wire Line
-	3500 5650 3000 5650
-Wire Wire Line
-	3500 5750 3000 5750
-Wire Wire Line
-	3500 5850 3000 5850
-Wire Wire Line
-	3500 5950 3000 5950
-Wire Wire Line
-	3500 6050 3000 6050
-Wire Wire Line
-	3000 6150 3500 6150
-Wire Wire Line
-	3500 6250 3000 6250
-Wire Wire Line
-	3500 6350 3000 6350
-Wire Wire Line
-	3500 6450 3000 6450
 Text HLabel 950  3200 0    50   BiDi ~ 0
 WAKE
@@
 Wire Wire Line
 	3300 2250 3350 2250
-Wire Wire Line
-	1500 3200 1650 3200
-Wire Wire Line
-	950  3200 1650 3200
 $Comp
 L power:PWR_FLAG #FLG0103
@@
 Wire Wire Line
 	3250 2500 3250 2900
+Wire Wire Line
+	1500 3200 1650 3200
+Wire Wire Line
+	950  3200 1650 3200
+NoConn ~ 4250 3500
+NoConn ~ 4250 3800
+NoConn ~ 4250 3900
+NoConn ~ 4250 4000
+NoConn ~ 2550 3700
+NoConn ~ 2550 3800
+NoConn ~ 2550 3900
+NoConn ~ 2550 3500
+NoConn ~ 2550 3400
+NoConn ~ 2550 3300
 $EndSCHEMATC

Commit message: ultima version
Parts:
- C57: value 100 nF -> 0.1nF
- C58: value 100 nF -> 0.1uF
- R1: value 100 K -> 100K
Connections:
- net Earth: no longer MOD1.12 (GND), MOD1.13 (GND), MOD1.15 (GND), MOD1.16 (GND), MOD1.2 (GND), MOD1.23 (GND), MOD1.24 (GND), MOD1.31 (GND), MOD1.32 (GND), MOD1.33 (GND), MOD1.34 (GND)
Changed lines of the file:
@@
-EESchema Schematic File Version 5
+EESchema Schematic File Version 4
 LIBS:Embebidos_2019-cache
 EELAYER 29 0
@@
 NoConn ~ 2550 3100
 NoConn ~ 2550 3600
-Wire Wire Line
-	2750 4400 2850 4400
-Wire Wire Line
-	2950 4400 3050 4400
-Wire Wire Line
-	3150 4400 3250 4400
-Wire Wire Line
-	3350 4400 3450 4400
-Wire Wire Line
-	3550 4400 3650 4400
-Wire Wire Line
-	3750 4400 3850 4400
-Wire Wire Line
-	3950 4400 4050 4400
-Wire Wire Line
-	2850 4400 2950 4400
-Connection ~ 2850 4400
-Connection ~ 2950 4400
-Wire Wire Line
-	3050 4400 3150 4400
-Connection ~ 3050 4400
-Connection ~ 3150 4400
-Wire Wire Line
-	3250 4400 3350 4400
-Connection ~ 3250 4400
 Connection ~ 3350 4400
-Wire Wire Line
-	3450 4400 3550 4400
-Connection ~ 3450 4400
-Connection ~ 3550 4400
-Wire Wire Line
-	3650 4400 3750 4400
-Connection ~ 3650 4400
-Connection ~ 3750 4400
-Wire Wire Line
-	3850 4400 3950 4400
-Connection ~ 3850 4400
-Connection ~ 3950 4400
 $Comp
 L power:Earth #PWR02
@@
 P 1650 3350
 F 0 "R1" H 1580 3304 50  0000 R CNN
-F 1 "100 K" H 1580 3395 50  0000 R CNN
+F 1 "100K" H 1580 3395 50  0000 R CNN
 F 2 "Embebidos_2019:R_0603_1608Metric_Pad1.05x0.95mm_HandSolder" V 1580 3350 50  0001 C CNN
 F 3 "~" H 1650 3350 50  0001 C CNN
@@
 	-1   0    0    1
 $EndComp
-Wire Wire Line
-	2550 3200 1650 3200
 $Comp
 L power:Earth #PWR01
@@
 P 3950 2700
 F 0 "C58" V 3698 2700 50  0000 C CNN
-F 1 "100 nF" V 3789 2700 50  0000 C CNN
+F 1 "0.1uF" V 3789 2700 50  0000 C CNN
 F 2 "Embebidos_2019:C_0603_1608Metric_Pad1.05x0.95mm_HandSolder" H 3988 2550 50  0001 C CNN
 F 3 "~" H 3950 2700 50  0001 C CNN
@@
 P 3950 2250
 F 0 "C57" V 3698 2250 50  0000 C CNN
-F 1 "100 nF" V 3789 2250 50  0000 C CNN
+F 1 "0.1nF" V 3789 2250 50  0000 C CNN
 F 2 "Embebidos_2019:C_0603_1608Metric_Pad1.05x0.95mm_HandSolder" H 3988 2100 50  0001 C CNN
 F 3 "~" H 3950 2250 50  0001 C CNN
@@
 NoConn ~ 2550 3300
 Wire Wire Line
-	1500 3200 1650 3200
-Wire Wire Line
-	950  3200 1650 3200
+	950  3200 2550 3200
+Wire Wire Line
+	2750 4400 3350 4400
+Wire Wire Line
+	3350 4400 4050 4400
 $EndSCHEMATC
