File: Embebidos_2019/Embebidos_2019.kicad_pcb (KiCad board)
At the start: 2 copper layers, 118 parts, among them CON1 SJ-3523-SMT-TR, J1 A106614-ND, J2 A128518-ND, J3 USB_A, J4 Barrel_Jack_Switch, J5 Conn_01x14_Male, SW1 SW_Push, U1 ADS1292R-TQFP, U2 OMEGA_2, U3 ZLDO1117G33TA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

Commit message: Add files via upload
Parts:
- removed C25: 0.1uF, Embebidos_2019:C_0603_1608Metric_Pad1.05x0.95mm_HandSolder
- removed C38: 1nF, Embebidos_2019:C_0603_1608Metric_Pad1.05x0.95mm_HandSolder
- BT1: moved to B.Cu
- J1: footprint Connector_PinSocket_2.54mm:PinSocket_1x12_P2.54mm_Vertical -> Connector_PinHeader_2.54mm:PinHeader_2x06_P2.54mm_Vertical
- J2: footprint Connector_PinSocket_2.54mm:PinSocket_1x03_P2.54mm_Vertical -> Connector_PinHeader_2.54mm:PinHeader_1x03_P2.54mm_Vertical
- J5: footprint Connector_PinHeader_1.27mm:PinHeader_1x14_P1.27mm_Vertical -> Connector_PinHeader_2.54mm:PinHeader_2x07_P2.54mm_Vertical
- moved C22 328.4 mm to (350.0, 115.1)
- moved C23 328.4 mm to (350.0, 110.0)
- moved R19 328.4 mm to (350.0, 90.9)
- moved SW1 328.4 mm to (357.6, 79.5)
- moved R1 218.0 mm to (316.2, 50.7)
- moved R17 217.1 mm to (275.8, 68.8)
- moved C24 216.7 mm to (279.9, 83.2)
- moved C26 216.7 mm to (242.4, 85.7)
- moved C57 216.7 mm to (313.9, 62.7)
- moved C58 216.7 mm to (308.4, 64.8)
- moved D1 216.7 mm to (279.9, 88.9)
- moved D2 216.7 mm to (287.5, 88.9)
- moved L2 216.7 mm to (293.2, 93.3)
- moved R16 216.7 mm to (275.5, 73.7)
- moved R18 216.7 mm to (275.5, 64.1)
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Connections:
- net /OMEGA2/JTAG_OM0 renamed /OMEGA2/JTAGOM0
- net /OMEGA2/JTAG_OM1 renamed /OMEGA2/JTAGOM1
- net /OMEGA2/JTAG_OM2 renamed /OMEGA2/JTAGOM2
- net /OMEGA2/JTAG_OM4 renamed /OMEGA2/JTAGOM4
- net /OMEGA2/JTAG_OM5 renamed /OMEGA2/JTAGOM5
- net /OMEGA2/TDO renamed /OMEGA2/JTAGOM3
- net /STM32/I2C1_SCL renamed /STM32/I2C1_U0
- net /STM32/I2C_U1 renamed /STM32/I2C1_U1
- net /STM32/TCK renamed /STM32/JTAG1
- net /STM32/TRST renamed /STM32/JTAG4
- C22 pad 1: +3.3V_MCU -> +3.3V_OM
- C23 pad 1: +3.3V_MCU -> +3.3V_OM
- R14 pad 2: /OMEGA2/SPI_OM_0 -> /OMEGA2/MOSI
- R15 pad 2: /OMEGA2/SPI_OM_1 -> /STM32/SPI2_U1
- R16 pad 2: /OMEGA2/SPI_OM_0 -> /STM32/SPI2_U0
- R17 pad 2: /OMEGA2/SPI_OM_2 -> /STM32/SPI2_U2
- R18 pad 2: /OMEGA2/SPI_CS -> /STM32/SPI2_U3
- R19 pad 2: +3.3V_MCU -> +3.3V_OM
- U1 pad 19: /ADS1292R/SPI_MOSI -> /ADS1292R/SPI_ADS0
- U2 pad 31: +3.3V_MCU -> +3.3V_OM
- U6 pad 20: /STM32/SPI1_NSS -> /ADS1292R/SPI_ADS3
- U6 pad 21: /STM32/SPI1_U2 -> /ADS1292R/SPI_ADS2
- U6 pad 22: /STM32/SPI1_MISO -> /ADS1292R/SPI_ADS1
- U6 pad 23: /STM32/SPI1_U0 -> /ADS1292R/SPI_ADS0
- U6 pad 36: /STM32/SPI2_MOSI -> /STM32/SPI2_U0
- U6 pad 7: /STM32/NRST -> /STM32/JTAG5
Routing:
- net Earth: track 0.00 -> 216.9 mm, vias 0 -> 5
- net +3.3V_MCU: track 0.00 -> 84.7 mm, vias 0 -> 2
- net /SUPPLY/AVSS: track 0.00 -> 44.3 mm
- net +3.3V_OM: track 0.00 -> 41.6 mm, vias 0 -> 2
- net +5V: track 0.00 -> 39.2 mm
- net /ADS1292R/AVDD: track 0.00 -> 31.8 mm, vias 0 -> 2
- net Net-(C15-Pad1): track 0.00 -> 25.9 mm
- net /STM32/PC3: track 0.00 -> 23.6 mm, vias 0 -> 2
- net /STM32/PC1: track 0.00 -> 23.1 mm, vias 0 -> 2
- net /STM32/PC2: track 0.00 -> 23.1 mm, vias 0 -> 2
- net /STM32/JTAG5: track 0.00 -> 23.0 mm, vias 0 -> 2
- net Net-(C13-Pad2): track 0.00 -> 22.9 mm, vias 0 -> 2
- net /STM32/PC0: track 0.00 -> 22.9 mm, vias 0 -> 2
- net Net-(C13-Pad1): track 0.00 -> 22.0 mm, vias 0 -> 2
- net /ADS1292R/IN2N: track 0.00 -> 20.9 mm, vias 0 -> 2
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Other:
- rule via_min_size: 0.4 -> 0.5

Commit message: los archivos ya fueron modificados
Parts:
- moved SW1 296.4 mm to (63.0, 111.8)
- moved R19 284.4 mm to (66.0, 107.2), turned to 0 degrees
- moved C22 275.9 mm to (80.6, 55.2), turned to 270 degrees
- moved C23 271.8 mm to (83.8, 55.2), turned to 270 degrees
- moved R32 260.8 mm to (47.8, 72.6), turned to 90 degrees
- moved D2 260.6 mm to (26.9, 92.5), turned to 180 degrees
- moved L1 260.0 mm to (34.0, 98.6), turned to 180 degrees
- moved R31 257.6 mm to (47.8, 68.6)
- moved D1 255.2 mm to (24.9, 99.1), turned to 180 degrees
- moved L2 255.1 mm to (38.1, 92.8), turned to 270 degrees
- moved R21 254.9 mm to (32.0, 94.0), turned to 270 degrees
- moved R20 244.9 mm to (35.1, 94.0), turned to 270 degrees
- moved C24 242.2 mm to (38.1, 97.8), turned to 270 degrees
- moved R1 222.6 mm to (96.5, 86.4)
- moved C57 214.5 mm to (100.3, 82.5)
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Routing:
- net Earth: track 216.9 -> 379.3 mm
- net Net-(C24-Pad1): track 0.00 -> 26.0 mm, vias 0 -> 2
- net Net-(D2-Pad2): track 0.00 -> 21.5 mm, vias 0 -> 2
- net Net-(D2-Pad1): track 0.00 -> 16.7 mm
- net /OMEGA2/RST_BTN: track 0.00 -> 11.7 mm
- net Net-(J2-Pad3): track 0.00 -> 11.3 mm
- net Net-(J2-Pad2): track 0.00 -> 11.1 mm
- net +3.3V_MCU: track 84.7 -> 91.5 mm
- net +3.3V_OM: track 41.6 -> 48.3 mm
- net /OMEGA2/BOOT0: track 0.00 -> 4.14 mm
- net Net-(R18-Pad1): track 0.00 -> 4.12 mm
- net Net-(L1-Pad3): track 0.00 -> 3.65 mm
- net Net-(R17-Pad1): track 0.00 -> 3.63 mm
- net Net-(R15-Pad1): track 0.00 -> 3.34 mm
- net Net-(R16-Pad1): track 0.00 -> 3.15 mm
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
Commit message: Add files via upload
Parts:
- removed J1: A106614-ND, Connector_PinHeader_2.54mm:PinHeader_2x06_P2.54mm_Vertical
- added C25: 0.1uF, Embebidos_2019:C_0603_1608Metric_Pad1.05x0.95mm_HandSolder, F.Cu at (95.5, 121.2)
- added C38: 1nF, Embebidos_2019:C_0603_1608Metric_Pad1.05x0.95mm_HandSolder, F.Cu at (93.3, 30.8)
- C28, C32, C35, D2, U3: moved to B.Cu
- moved FB1 129.7 mm to (72.3, 76.4), turned to 90 degrees
- moved C1 126.8 mm to (70.1, 66.0), turned to 270 degrees
- moved R9 122.8 mm to (76.8, 79.4), turned to 90 degrees
- moved C2 121.4 mm to (72.9, 66.1), turned to 270 degrees
- moved C5 115.9 mm to (75.7, 66.0), turned to 270 degrees
- moved C40 114.5 mm to (89.6, 38.4), turned to 90 degrees
- moved C14 114.0 mm to (80.5, 77.3), turned to 270 degrees
- moved C41 113.4 mm to (88.4, 43.7), turned to 180 degrees
- moved C8 110.4 mm to (78.5, 66.0), turned to 270 degrees
- moved C42 109.8 mm to (89.3, 47.6), turned to 270 degrees
- moved C39 109.0 mm to (92.5, 38.4), turned to 90 degrees
- moved R6 108.5 mm to (83.5, 77.3), turned to 90 degrees
- moved L3 106.0 mm to (92.6, 42.8), turned to 270 degrees
- moved R26 103.8 mm to (55.5, 39.0)
- moved C37 103.7 mm to (96.3, 36.5), turned to 0 degrees
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Connections:
- C49 pad 1: /STM32/NRST -> /STM32/JTAG5
- MOD1 pad 14: /BLUETOOTH/PIO7 -> Net-(MOD1-Pad14)
- MOD1 pad 19: /BLUETOOTH/PIO8 -> Net-(MOD1-Pad19)
- MOD1 pad 26: /BLUETOOTH/PIO9 -> Net-(MOD1-Pad26)
- MOD1 pad 28: /BLUETOOTH/PIO10 -> Net-(MOD1-Pad28)
- MOD1 pad 29: /BLUETOOTH/PIO11 -> Net-(MOD1-Pad29)
- MOD1 pad 3: /BLUETOOTH/AIO2 -> Net-(MOD1-Pad3)
- MOD1 pad 4: /BLUETOOTH/AIO1 -> Net-(MOD1-Pad4)
- MOD1 pad 5: /BLUETOOTH/AIO0 -> Net-(MOD1-Pad5)
- MOD1 pad 8: /BLUETOOTH/PIO3 -> Net-(MOD1-Pad8)
- MOD1 pad 9: /BLUETOOTH/PIO4 -> Net-(MOD1-Pad9)
- R14 pad 2: /OMEGA2/MOSI -> /STM32/SPI1_U0
- R15 pad 2: /STM32/SPI2_U1 -> /STM32/SPI1_U1
- R16 pad 2: /STM32/SPI2_U0 -> /STM32/SPI1_U0
- R17 pad 2: /STM32/SPI2_U2 -> /STM32/SPI1_U2
- R18 pad 2: /STM32/SPI2_U3 -> /STM32/SPI1_U3
- R28 pad 2: /STM32/NRST -> /STM32/JTAG5
- S1 pad 1: /STM32/NRST -> /STM32/JTAG5
- S1 pad 2: /STM32/NRST -> /STM32/JTAG5
- U2 pad 2: /OMEGA2/JTAGOM0 -> /STM32/JTAG0
- U2 pad 3: /OMEGA2/JTAGOM1 -> /STM32/JTAG1
- U2 pad 4: /OMEGA2/JTAGOM2 -> /STM32/JTAG2
- U2 pad 5: /OMEGA2/JTAGOM3 -> /STM32/JTAG3
- U2 pad 6: /OMEGA2/JTAGOM4 -> /STM32/JTAG4
- U2 pad 7: /OMEGA2/JTAGOM5 -> /STM32/JTAG5
- U6 pad 20: /ADS1292R/SPI_ADS3 -> /STM32/SPI1_U3
- U6 pad 21: /ADS1292R/SPI_ADS2 -> /STM32/SPI1_U2
- U6 pad 22: /ADS1292R/SPI_ADS1 -> /STM32/SPI1_U1
- U6 pad 23: /ADS1292R/SPI_ADS0 -> /STM32/SPI1_U0
- U6 pad 26: /STM32/A_PWDN -> /STM32/PC6
- U6 pad 33: /STM32/SPI2_U3 -> /ADS1292R/SPI_ADS3
- U6 pad 34: /STM32/SPI2_U2 -> /ADS1292R/SPI_ADS2
- U6 pad 35: /STM32/SPI2_U1 -> /ADS1292R/SPI_ADS1
- U6 pad 36: /STM32/SPI2_U0 -> /ADS1292R/SPI_ADS0
- U6 pad 37: /STM32/PC6 -> /STM32/A_CLK
- U6 pad 38: /STM32/PC7 -> /STM32/A_START
- U6 pad 39: /STM32/PC8 -> /STM32/A_PWDN
- U6 pad 40: /STM32/PC9 -> /STM32/A_CLKSEL
- U6 pad 41: /STM32/A_CLKSEL -> /STM32/PC7
- U6 pad 42: /STM32/A_CLK -> /STM32/PC8
- U6 pad 43: /STM32/A_START -> /STM32/PC9
- U6 pad 55: /STM32/TDO -> /STM32/JTAG3
- U6 pad 61: /STM32/I2C1_U0 -> /OMEGA2/I2C_OM0
- U6 pad 62: /STM32/I2C1_U1 -> /OMEGA2/I2C_OM1
Routing:
- net /OMEGA2/I2C_OM0: track 0.00 -> 112.6 mm
- net /OMEGA2/I2C_OM1: track 0.00 -> 107.4 mm
- net /OMEGA2/BOOT0: track 4.14 -> 85.7 mm, vias 0 -> 2
- net /OMEGA2/BOOT1: track 9.73 -> 85.4 mm, vias 0 -> 1
- net /STM32/PC7: track 0.00 -> 67.1 mm, vias 0 -> 2
- net /STM32/PC8: track 0.00 -> 67.1 mm, vias 0 -> 2
- net /STM32/PC9: track 0.00 -> 63.5 mm, vias 0 -> 2
- net +5V: track 39.2 -> 101.9 mm, vias 0 -> 3
- net Net-(BT1-Pad1): track 0.00 -> 59.9 mm, vias 0 -> 1
- net /STM32/JTAG5: track 23.0 -> 69.5 mm, vias 2 -> 3
- net /STM32/JTAG2: track 0.00 -> 44.9 mm, vias 0 -> 2
- net /STM32/JTAG4: track 0.00 -> 44.3 mm, vias 0 -> 2
- net Net-(CON1-Pad1): track 0.00 -> 41.9 mm, vias 0 -> 2
- net /STM32/JTAG0: track 0.00 -> 41.7 mm, vias 0 -> 1
- net /STM32/JTAG1: track 0.00 -> 41.3 mm, vias 0 -> 2
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
Commit message: los archivos ya fueron modificados, por fin  subio
Connections:
- net /ADS1292R/SPI_ADS0 renamed /STM32/SPI2_U0
- net /ADS1292R/SPI_ADS1 renamed /STM32/SPI2_U1
- net /ADS1292R/SPI_ADS2 renamed /STM32/SPI2_U2
- net /ADS1292R/SPI_ADS3 renamed /STM32/SPI2_U3
- net /STM32/A_CLK renamed /ADS1292R/ADS_CLK
- net /STM32/A_CLKSEL renamed /ADS1292R/ADS_CLKSEL
- net /STM32/A_DRY renamed /ADS1292R/ADS_DRDY
- net /STM32/A_PWDN renamed /ADS1292R/ADS_PWDN
- net /STM32/A_START renamed /ADS1292R/ADS_START
- C42 pad 2: /SUPPLY/AVSS -> /ADS1292R/AVSS
- J5 pad 10: /STM32/PC6 -> /STM32/PC3
- J5 pad 11: /STM32/PC7 -> /STM32/PC10
- J5 pad 12: /STM32/PC8 -> /STM32/PC7
- J5 pad 14: /STM32/PC10 -> /STM32/PC8
- J5 pad 5: /STM32/PC1 -> /STM32/PC4
- J5 pad 6: /STM32/PC2 -> /STM32/PC1
- J5 pad 7: /STM32/PC3 -> /STM32/PC5
- J5 pad 8: /STM32/PC4 -> /STM32/PC2
- J5 pad 9: /STM32/PC5 -> /STM32/PC6
- R20 pad 2: Net-(L1-Pad2) -> Net-(R20-Pad2)
- R21 pad 2: Net-(L1-Pad3) -> Net-(R21-Pad2)
- R26 pad 2: Net-(BT1-Pad1) -> Net-(R26-Pad2)
- R29 pad 2: Net-(D4-Pad1) -> Net-(R29-Pad2)
- R30 pad 2: Net-(D5-Pad1) -> Net-(R30-Pad2)
- U1 pad 1: Net-(C11-Pad1) -> Net-(U1-Pad1)
- U1 pad 10: /SUPPLY/AVSS -> /ADS1292R/AVSS
- U1 pad 11: Net-(C6-Pad1) -> Net-(U1-Pad11)
- U1 pad 13: /SUPPLY/AVSS -> /ADS1292R/AVSS
- U1 pad 2: Net-(C11-Pad2) -> Net-(U1-Pad2)
- U1 pad 27: Net-(C10-Pad1) -> Net-(U1-Pad27)
- U1 pad 28: Net-(C14-Pad1) -> Net-(U1-Pad28)
- U1 pad 29: Net-(R5-Pad2) -> Net-(U1-Pad29)
- U1 pad 3: Net-(C15-Pad1) -> Net-(U1-Pad3)
- U1 pad 30: Net-(R2-Pad2) -> Net-(U1-Pad30)
- U1 pad 31: Net-(R11-Pad2) -> Net-(U1-Pad31)
- U1 pad 32: Net-(R10-Pad2) -> Net-(U1-Pad32)
- U1 pad 4: Net-(C13-Pad1) -> Net-(U1-Pad4)
- U1 pad 7: Net-(C12-Pad1) -> Net-(U1-Pad7)
- U1 pad 8: Net-(C12-Pad2) -> Net-(U1-Pad8)
- U1 pad 9: Net-(C3-Pad1) -> Net-(U1-Pad9)
- U6 pad 17: /OMEGA2/USART_TX -> /STM32/UART2_RX
- U6 pad 45: /STM32/UART_RTS -> /BLUETOOTH/Bluetooth_CTS
- U6 pad 58: /STM32/UART1_TX -> /BLUETOOTH/Bluetooth_RX
- U6 pad 61: /OMEGA2/I2C_OM0 -> /STM32/I2C1_U0
- U6 pad 62: /OMEGA2/I2C_OM1 -> /STM32/I2C1_U1
Routing:
- net +3.3V_MCU: track 108.5 -> 203.1 mm, vias 4 -> 9
- net +5V: track 101.9 -> 160.8 mm, vias 3 -> 5
- net +3.3V_OM: track 51.2 -> 92.1 mm
- net /STM32/PC3: track 37.2 -> 69.3 mm
- net /STM32/PC2: track 36.0 -> 64.4 mm
- net /STM32/PC1: track 35.2 -> 60.0 mm
- net /STM32/PC0: track 36.2 -> 55.0 mm
- net /STM32/PC4: track 34.3 -> 47.5 mm
- net /STM32/PC7: track 67.1 -> 78.2 mm
- net /STM32/PC5: track 35.5 -> 46.5 mm
- net /STM32/PC6: track 32.6 -> 42.8 mm
- net /STM32/PC10: track 17.7 -> 25.5 mm
- net /STM32/PC9: track 63.5 -> 71.3 mm
- net /STM32/PC8: track 67.1 -> 73.2 mm
- net /ADS1292R/AVDD: track 35.7 -> 41.3 mm, vias 3 -> 4
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
Commit message: Bueno esto casi me saca canas, esta es la ultima version ya puedes editar
Connections:
- R26 pad 2: Net-(R26-Pad2) -> Net-(BT1-Pad1)
- U6 pad 17: /STM32/UART2_RX -> /OMEGA2/USART_TX
- U6 pad 45: /BLUETOOTH/Bluetooth_CTS -> /STM32/UART_RTS
Routing:
- net +3.3V_MCU: track 203.1 -> 200.6 mm, vias 9 -> 8
- net +5V: vias 5 -> 4
- added copper zone on B.Cu, net Earth
- added copper zone on F.Cu, net Earth

Commit message: Add files via upload
Parts:
- moved R22 0.12 mm to (95.5, 42.9)
Connections:
- net /ADS1292R/ADS_CLK renamed /STM32/A_CLK
- net /ADS1292R/ADS_CLKSEL renamed /STM32/A_CLKSEL
- net /ADS1292R/ADS_DRDY renamed /STM32/A_DRY
- net /ADS1292R/ADS_PWDN renamed /STM32/A_PWDN
- net /ADS1292R/ADS_START renamed /STM32/A_START
- net /STM32/SPI2_U0 renamed /ADS1292R/SPI_ADS0
- net /STM32/SPI2_U1 renamed /ADS1292R/SPI_ADS1
- net /STM32/SPI2_U2 renamed /ADS1292R/SPI_ADS2
- net /STM32/SPI2_U3 renamed /ADS1292R/SPI_ADS3
- C42 pad 2: /ADS1292R/AVSS -> /SUPPLY/AVSS
- R20 pad 2: Net-(R20-Pad2) -> Net-(L1-Pad2)
- R21 pad 2: Net-(R21-Pad2) -> Net-(L1-Pad3)
- R29 pad 2: Net-(R29-Pad2) -> Net-(D4-Pad1)
- R30 pad 2: Net-(R30-Pad2) -> Net-(D5-Pad1)
- U1 pad 1: Net-(U1-Pad1) -> Net-(C11-Pad1)
- U1 pad 10: /ADS1292R/AVSS -> /SUPPLY/AVSS
- U1 pad 11: Net-(U1-Pad11) -> Net-(C6-Pad1)
- U1 pad 13: /ADS1292R/AVSS -> /SUPPLY/AVSS
- U1 pad 2: Net-(U1-Pad2) -> Net-(C11-Pad2)
- U1 pad 27: Net-(U1-Pad27) -> Net-(C10-Pad1)
- U1 pad 28: Net-(U1-Pad28) -> Net-(C14-Pad1)
- U1 pad 29: Net-(U1-Pad29) -> Net-(R5-Pad2)
- U1 pad 3: Net-(U1-Pad3) -> Net-(C15-Pad1)
- U1 pad 30: Net-(U1-Pad30) -> Net-(R2-Pad2)
- U1 pad 31: Net-(U1-Pad31) -> Net-(R11-Pad2)
- U1 pad 32: Net-(U1-Pad32) -> Net-(R10-Pad2)
- U1 pad 4: Net-(U1-Pad4) -> Net-(C13-Pad1)
- U1 pad 7: Net-(U1-Pad7) -> Net-(C12-Pad1)
- U1 pad 8: Net-(U1-Pad8) -> Net-(C12-Pad2)
- U1 pad 9: Net-(U1-Pad9) -> Net-(C3-Pad1)
- U6 pad 58: /BLUETOOTH/Bluetooth_RX -> /STM32/UART1_TX
- U6 pad 61: /STM32/I2C1_U0 -> /OMEGA2/I2C_OM0
- U6 pad 62: /STM32/I2C1_U1 -> /OMEGA2/I2C_OM1
Routing:
- net Earth: track 368.8 -> 411.0 mm, vias 4 -> 14
- net Net-(BT1-Pad1): track 59.9 -> 93.4 mm
- net +3.3V_OM: track 92.1 -> 93.2 mm

Commit message: ultima version
Routing:
- net +5V: track 160.8 -> 178.6 mm
- net Earth: track 411.0 -> 405.4 mm, vias 14 -> 275
Other:
- board outline added: 99.5 x 99.1 mm
