File: Embebidos_2019/SUPPLY.sch (KiCad schematic (older format))
At the start: 25 parts, among them J4 Barrel_Jack_Switch, U3 ZLDO1117G33TA, U4 ZLDO1117G33TA, U5 TPS73201

Commit message: Add files via upload
Changed lines of the file:
@@
-	1    0    0    -1
-$EndComp
-$Comp
-L Embebidos_2019-rescue:+5V-power-pcb_embedded_systems-rescue #PWR?
-U 1 1 5C91E97D
-P 6950 1400
-AR Path="/5C91E97D" Ref="#PWR?"  Part="1"
-AR Path="/5CE6DB76/5C91E97D" Ref="#PWR031"  Part="1"
-F 0 "#PWR031" H 6950 1250 50  0001 C CNN
-F 1 "+5V" H 6965 1573 50  0000 C CNN
-F 2 "" H 6950 1400 50  0001 C CNN
-F 3 "" H 6950 1400 50  0001 C CNN
-	1    6950 1400
 	1    0    0    -1
 $EndComp
@@
 Wire Notes Line
 	6300 2300 6300 1150
-Wire Notes Line
-	6300 1150 7250 1150
 Wire Notes Line
 	7250 1150 7250 2300
@@
 Wire Wire Line
 	6950 2050 6950 2000
+Text GLabel 6900 1250 0    50   Input ~ 0
++5V
+Wire Wire Line
+	6950 1400 6950 1250
+Wire Wire Line
+	6950 1250 6900 1250
+$Comp
+L power:PWR_FLAG #FLG0108
+U 1 1 5CF05EA9
+P 3400 8350
+F 0 "#FLG0108" H 3400 8425 50  0001 C CNN
+F 1 "PWR_FLAG" H 3400 8523 50  0000 C CNN
+F 2 "" H 3400 8350 50  0001 C CNN
+F 3 "~" H 3400 8350 50  0001 C CNN
+	1    3400 8350
+	1    0    0    -1
+$EndComp
+Wire Wire Line
+	3400 8350 3400 8550
 $EndSCHEMATC

Commit message: los archivos ya fueron modificados, por fin  subio
Connections:
- net at C39.1, C40.1, L3.1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: no longer R22.1
Changed lines of the file:
@@
-EESchema Schematic File Version 5
+EESchema Schematic File Version 4
 LIBS:Embebidos_2019-cache
 EELAYER 29 0
@@
 $EndComp
 Wire Wire Line
-	5000 8550 4350 8550
-Wire Wire Line
 	5000 8850 4600 8850
 Wire Wire Line
@@
 $EndComp
 Wire Wire Line
-	5450 8550 5000 8550
-Connection ~ 5000 8550
-Wire Wire Line
 	5900 8550 5450 8550
 Connection ~ 5450 8550
@@
 Wire Wire Line
 	3400 8350 3400 8550
+Wire Wire Line
+	4350 8550 5450 8550
 $EndSCHEMATC

Commit message: Add files via upload
Connections:
- net at C39.1, C40.1, L3.1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: now also R22.1
Changed lines of the file:
@@
-EESchema Schematic File Version 4
+EESchema Schematic File Version 5
 LIBS:Embebidos_2019-cache
 EELAYER 29 0
@@
 	3400 8350 3400 8550
 Wire Wire Line
-	4350 8550 5450 8550
+	4350 8550 5000 8550
+Connection ~ 5000 8550
+Wire Wire Line
+	5000 8550 5450 8550
 $EndSCHEMATC

Commit message: ultima version
Connections:
- net at C39.1, C40.1, L3.1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: no longer R22.1
Changed lines of the file:
@@
-EESchema Schematic File Version 5
+EESchema Schematic File Version 4
 LIBS:Embebidos_2019-cache
 EELAYER 29 0
@@
 	3400 8350 3400 8550
 Wire Wire Line
-	4350 8550 5000 8550
-Connection ~ 5000 8550
-Wire Wire Line
-	5000 8550 5450 8550
+	4350 8550 5450 8550
 $EndSCHEMATC
